File: pcb/verasity/verasity_PCB/verasity_PCB.kicad_pcb (KiCad board)
At the start: 2 copper layers, 342.9 x 119.1 mm, 110 parts, among them U10 F7, U11 F8, U12 F9, U13 F10, U14 F11, U15 F12, U16 PR_SC, U17 SCRLC, U18 PoBr, U19 `, U2 ESC, U20 1, U21 2, U22 3, U23 4, U24 5, U25 6, U26 7, U27 8, U28 9, U29 0, U3 custom1, U30 -, U31 =, U32 BackSp, U33 Ins, U34 Home, U35 PaUp, U36 Tab, U37 Q, U38 W, U39 E, U4 F1, U40 R, U41 T, U42 Y, U43 U, U44 I, U45 O, U46 P, U47 [, U48 ], U49 \, U5 F2, U50 Del, U51 End, U52 PaDo, U53 Caps, U54 A, U55 S, U56 D, U57 F, U58 G, U59 H, U6 F3, U60 J, U61 K, U62 L, U63 ;, U64 ", U65 Ent, U66 LShif, U67 Z, U68 X, U69 C, U7 F4, U70 V, U71 B, U72 N, U73 M, U74 <, U75 >, U76 ?, U77 Custom, U78 RShif, U79 ArUp, U8 F5, U80 LCrtl, U81 LSuper, U82 LAlt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

Commit message: cc
Signed-off-by: bornav <borna.vincek1@gmail.com>
Changed lines of the file:
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@@
     (tags "mounting hole 2.2mm no annular m2")
     (attr exclude_from_pos_files exclude_from_bom)
-    (fp_text reference "REF**" (at 0 -3.2) (layer "F.SilkS") hide
+    (fp_text reference "REF**" (at 0 -3.2) (layer "F.SilkS")
         (effects (font (size 1 1) (thickness 0.15)))
     )
@@
     (tags "mounting hole 2.2mm no annular m2")
     (attr exclude_from_pos_files exclude_from_bom)
-    (fp_text reference "REF**" (at 0 -3.2) (layer "F.SilkS") hide
+    (fp_text reference "REF**" (at 0 -3.2) (layer "F.SilkS")
         (effects (font (size 1 1) (thickness 0.15)))
     )
@@
     (tags "mounting hole 2.2mm no annular m2")
     (attr exclude_from_pos_files exclude_from_bom)
-    (fp_text reference "REF**" (at 0 -3.2) (layer "F.SilkS") hide
+    (fp_text reference "REF**" (at 0 -3.2) (layer "F.SilkS")
         (effects (font (size 1 1) (thickness 0.15)))
     )
@@
     (fp_circle (center 0 0) (end 2.45 0)
       (stroke (width 0.05) (type solid)) (fill none) (layer "F.CrtYd"))
-    (pad "" np_thru_hole circle (at 0 0) (size 2.2 2.2) (drill 2.2) (layers "F&B.Cu" "*.Mask"))
+    (pad "" np_thru_hole circle (at 0 0) (size 2.2 2.2) (drill 2.2) (layers "*.Cu" "*.Mask"))
   )
   (footprint "socket_multi_mechanical_keyboard:inverse_socket_MX_hotswap" (layer "F.Cu")
@@
     (tags "mounting hole 2.2mm no annular m2")
     (attr exclude_from_pos_files exclude_from_bom)
-    (fp_text reference "REF**" (at 0 -3.2) (layer "F.SilkS") hide
+    (fp_text reference "REF**" (at 0 -3.2) (layer "F.SilkS")
         (effects (font (size 1 1) (thickness 0.15)))
     )
@@
     (tags "mounting hole 2.2mm no annular m2")
     (attr exclude_from_pos_files exclude_from_bom)
-    (fp_text reference "REF**" (at 0 -3.2) (layer "F.SilkS") hide
+    (fp_text reference "REF**" (at 0 -3.2) (layer "F.SilkS")
         (effects (font (size 1 1) (thickness 0.15)))
     )
@@
     (tags "mounting hole 2.2mm no annular m2")
     (attr exclude_from_pos_files exclude_from_bom)
-    (fp_text reference "REF**" (at 0 -3.2) (layer "F.SilkS") hide
+    (fp_text reference "REF**" (at 0 -3.2) (layer "F.SilkS")
         (effects (font (size 1 1) (thickness 0.15)))
     )
@@
     (fp_circle (center 0 0) (end 2.45 0)
       (stroke (width 0.05) (type solid)) (fill none) (layer "F.CrtYd"))
-    (pad "" np_thru_hole circle (at 0 0) (size 2.2 2.2) (drill 2.2) (layers "F&B.Cu" "*.Mask"))
+    (pad "" np_thru_hole circle (at 0 0) (size 2.2 2.2) (drill 2.2) (layers "*.Cu" "*.Mask"))
   )
   (footprint "socket_multi_mechanical_keyboard:inverse_socket_MX_hotswap" (layer "F.Cu")
@@
     (tags "mounting hole 2.2mm no annular m2")
     (attr exclude_from_pos_files exclude_from_bom)
-    (fp_text reference "REF**" (at 0 -3.2) (layer "F.SilkS") hide
+    (fp_text reference "REF**" (at 0 -3.2) (layer "F.SilkS")
         (effects (font (size 1 1) (thickness 0.15)))
     )
@@
     (fp_circle (center 0 0) (end 2.45 0)
       (stroke (width 0.05) (type solid)) (fill none) (layer "F.CrtYd"))
-    (pad "" np_thru_hole circle (at 0 0) (size 2.2 2.2) (drill 2.2) (layers "F&B.Cu" "*.Mask"))
+    (pad "" np_thru_hole circle (at 0 0) (size 2.2 2.2) (drill 2.2) (layers "*.Cu" "*.Mask"))
   )
   (footprint "socket_multi_mechanical_keyboard:inverse_socket_MX_hotswap" (layer "F.Cu")
@@
     (tags "mounting hole 2.2mm no annular m2")
     (attr exclude_from_pos_files exclude_from_bom)
-    (fp_text reference "REF**" (at 0 -3.2) (layer "F.SilkS") hide
+    (fp_text reference "REF**" (at 0 -3.2) (layer "F.SilkS")
         (effects (font (size 1 1) (thickness 0.15)))
     )
@@
     (tags "mounting hole 2.2mm no annular m2")
     (attr exclude_from_pos_files exclude_from_bom)
-    (fp_text reference "REF**" (at 0 -3.2) (layer "F.SilkS") hide
+    (fp_text reference "REF**" (at 0 -3.2) (layer "F.SilkS")
         (effects (font (size 1 1) (thickness 0.15)))
     )
@@
     (fp_circle (center 0 0) (end 2.45 0)
       (stroke (width 0.05) (type solid)) (fill none) (layer "F.CrtYd"))
-    (pad "" np_thru_hole circle (at 0 0) (size 2.2 2.2) (drill 2.2) (layers "F&B.Cu" "*.Mask"))
+    (pad "" np_thru_hole circle (at 0 0) (size 2.2 2.2) (drill 2.2) (layers "*.Cu" "*.Mask"))
   )
   (footprint "socket_multi_mechanical_keyboard:inverse_socket_MX_hotswap" (layer "F.Cu")

Commit message: prerelease
Signed-off-by: bornav <borna.vincek1@gmail.com>
Parts:
- U99: footprint waveshare:waveshare-rp2040-zero_no_inner -> waveshare:waveshare-rp2040-pad_solder_with_cutout
- moved U99 0.45 mm to (10.9, -85.8)
Connections:
- U99 pad 2: unconnected-(U99-GPIO0-Pad2) -> COL7
- U99 pad 8: COL7 -> unconnected-(U99-GPIO6-Pad8)
Routing:
- net ROW2: track 449.3 -> 354.2 mm
- net ROW6: track 557.0 -> 480.5 mm
- net ROW4: track 486.9 -> 415.4 mm
- net COL3: track 402.3 -> 349.6 mm
- net ROW3: track 420.3 -> 368.0 mm, vias 0 -> 1
- net ROW1: track 517.2 -> 549.1 mm
- net COL7: track 528.4 -> 502.6 mm
- net COL2: track 251.9 -> 273.0 mm, vias 0 -> 1
- net COL6: track 432.0 -> 411.1 mm
- net COL8: track 514.2 -> 497.6 mm
- net COL1: track 253.8 -> 268.7 mm
- net ROW5: track 446.4 -> 439.8 mm, vias 2 -> 1
- net COL4: track 316.4 -> 314.0 mm
- net COL5: track 354.2 -> 353.6 mm
Other:
- board text added: "JLCJLCJLCJLC"

Commit message: new 2.1 prod
Parts:
- removed REF** (x3): Stabilizer_MX_2u, socket_multi_mechanical_keyboard:Stabilizer_MX_2u
- removed REF** (x9): MountingHole_2.2mm_M2, MountingHole:MountingHole_2.2mm_M2
- added H1: MountingHole_Pad, MountingHole:MountingHole_2.1mm, F.Cu at (12.7, 3.00)
- added H2: MountingHole_Pad, MountingHole:MountingHole_2.1mm, F.Cu at (14.3, -54.8)
- added H3: MountingHole_Pad, MountingHole:MountingHole_2.1mm, F.Cu at (78.6, -34.5)
- added H4: MountingHole_Pad, MountingHole:MountingHole_2.1mm, F.Cu at (273.1, 3.00)
- added H5: MountingHole_Pad, MountingHole:MountingHole_2.1mm, F.Cu at (130.8, 3.00)
- added H6: MountingHole_Pad, MountingHole:MountingHole_2.1mm, F.Cu at (-7.50, -106.5)
- added H7: MountingHole_Pad, MountingHole:MountingHole_2.1mm, F.Cu at (271.5, -53.6)
- added H8: MountingHole_Pad, MountingHole:MountingHole_2.1mm, F.Cu at (140.5, -72.6)
- added H9: MountingHole_Pad, MountingHole:MountingHole_2.1mm, F.Cu at (327.7, -106.5)
- U32, U65, U66: footprint socket_multi_mechanical_keyboard:inverse_socket_MX_hotswap -> socket_multi_mechanical_keyboard:inverse_socket_MX_hotswap_2.5U_stabilizers
Connections:
- U10 pad 1: COL5 -> COL9
- U11 pad 1: COL5 -> COL10
- U12 pad 1: COL6 -> COL11
- U13 pad 1: COL6 -> COL12
- U14 pad 1: COL7 -> COL13
- U15 pad 1: COL7 -> COL14
- U16 pad 1: COL7 -> COL15
- U17 pad 1: COL8 -> COL16
- U18 pad 1: COL8 -> COL17
- U20 pad 1: COL1 -> COL2
- U21 pad 1: COL2 -> COL3
- U22 pad 1: COL2 -> COL4
- U23 pad 1: COL3 -> COL5
- U24 pad 1: COL3 -> COL6
- U25 pad 1: COL4 -> COL7
- U26 pad 1: COL4 -> COL8
- U27 pad 1: COL5 -> COL9
- U28 pad 1: COL5 -> COL10
- U29 pad 1: COL6 -> COL11
- U3 pad 1: COL7 -> COL15
- U30 pad 1: COL6 -> COL12
- U31 pad 1: COL7 -> COL13
- U32 pad 1: COL7 -> COL14
- U33 pad 1: COL7 -> COL15
- U34 pad 1: COL8 -> COL16
- U35 pad 1: COL8 -> COL17
- U37 pad 1: COL1 -> COL2
- U38 pad 1: COL2 -> COL3
- U39 pad 1: COL2 -> COL4
- U4 pad 1: COL2 -> COL3
- U40 pad 1: COL3 -> COL5
- U41 pad 1: COL3 -> COL6
- U42 pad 1: COL4 -> COL7
- U43 pad 1: COL4 -> COL8
- U44 pad 1: COL5 -> COL9
- U45 pad 1: COL5 -> COL10
- U46 pad 1: COL6 -> COL11
- U47 pad 1: COL6 -> COL12
- U48 pad 1: COL7 -> COL13
- U49 pad 1: COL7 -> COL14
- U5 pad 1: COL2 -> COL4
- U50 pad 1: COL7 -> COL15
- U51 pad 1: COL8 -> COL16
- U52 pad 1: COL8 -> COL17
- U54 pad 1: COL1 -> COL2
- U55 pad 1: COL2 -> COL3
- U56 pad 1: COL2 -> COL4
- U57 pad 1: COL3 -> COL5
- U58 pad 1: COL3 -> COL6
- U59 pad 1: COL4 -> COL7
- U6 pad 1: COL3 -> COL5
- U60 pad 1: COL4 -> COL8
- U61 pad 1: COL5 -> COL9
- U62 pad 1: COL5 -> COL10
- U63 pad 1: COL6 -> COL11
- U64 pad 1: COL6 -> COL12
- U65 pad 1: COL7 -> COL13
- U67 pad 1: COL1 -> COL2
- U68 pad 1: COL2 -> COL3
- U69 pad 1: COL2 -> COL4
- U7 pad 1: COL3 -> COL6
- U70 pad 1: COL3 -> COL5
- U71 pad 1: COL3 -> COL6
- U72 pad 1: COL4 -> COL7
- U73 pad 1: COL4 -> COL8
- U74 pad 1: COL5 -> COL9
- U75 pad 1: COL5 -> COL10
- U76 pad 1: COL6 -> COL11
- U77 pad 1: COL6 -> COL12
- U78 pad 1: COL7 -> COL13
- U79 pad 1: COL8 -> COL16
- U8 pad 1: COL4 -> COL7
- U81 pad 1: COL1 -> COL2
- U82 pad 1: COL2 -> COL3
- U83 pad 1: COL2 -> COL4
- U84 pad 1: COL3 -> COL5
- U85 pad 1: COL3 -> COL6
- U86 pad 1: COL4 -> COL7
- U87 pad 1: COL4 -> COL8
- U88 pad 1: COL8 -> COL16
- U89 pad 1: COL5 -> COL9
- U9 pad 1: COL4 -> COL8
- U90 pad 1: COL5 -> COL10
- U91 pad 1: COL6 -> COL11
- U92 pad 1: COL6 -> COL12
- U93 pad 1: COL7 -> COL15
- U94 pad 1: COL8 -> COL16
- U95 pad 1: COL8 -> COL17
- U96 pad 1: COL8 -> COL17
- U97 pad 1: COL7 -> COL15
- U98 pad 1: COL8 -> COL17
- U99 pad 11: COL2 -> COL9
- U99 pad 12: ROW3 -> COL8
- U99 pad 13: ROW2 -> COL7
- U99 pad 14: unconnected-(U99-GPIO11-Pad14) -> COL6
- U99 pad 15: unconnected-(U99-GPIO12-Pad15) -> COL5
- U99 pad 16: COL1 -> COL4
- U99 pad 17: ROW5 -> COL3
- U99 pad 18: unconnected-(U99-GPIO15-Pad18) -> COL2
- U99 pad 2: COL7 -> COL17
- U99 pad 3: COL6 -> COL16
- U99 pad 38: COL3 -> ROW2
- U99 pad 39: ROW6 -> ROW3
- U99 pad 4: COL5 -> COL15
- U99 pad 40: unconnected-(U99-GPIO28_ADC2-Pad40) -> ROW4
- U99 pad 41: unconnected-(U99-GPIO29_ADC3-Pad41) -> ROW6
- U99 pad 5: COL4 -> COL14
- U99 pad 6: ROW1 -> COL13
- U99 pad 7: ROW4 -> COL12
- U99 pad 8: unconnected-(U99-GPIO6-Pad8) -> COL11
- U99 pad 9: COL8 -> COL10
Routing:
- net COL17: track 0.00 -> 389.0 mm
- net COL16: track 0.00 -> 370.3 mm
- net COL12: track 0.00 -> 360.9 mm
- net COL15: track 0.00 -> 353.3 mm
- net COL11: track 0.00 -> 340.4 mm
- net COL13: track 0.00 -> 338.4 mm
- net COL10: track 0.00 -> 309.8 mm
- net COL9: track 0.00 -> 288.6 mm
- net COL14: track 0.00 -> 283.6 mm
- net COL7: track 502.6 -> 245.8 mm
- net COL8: track 497.6 -> 269.9 mm
- net COL6: track 411.1 -> 218.4 mm
- net COL3: track 349.6 -> 181.2 mm
- net COL2: track 273.0 -> 113.1 mm, vias 1 -> 0
- net COL5: track 353.6 -> 201.3 mm
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Other:
- board text added: "Verasity 2.1"
- board text removed: "Verasity 2.0"
