File: pcb/verasity/verasity_PCB/verasity_PCB.kicad_sch (KiCad schematic)
At the start: 98 parts, among them U10 F7, U11 F8, U12 F9, U13 F10, U14 F11, U15 F12, U16 PR_SC, U17 SCRLC, U18 PoBr, U19 `, U2 ESC, U20 1, U21 2, U22 3, U23 4, U24 5, U25 6, U26 7, U27 8, U28 9, U29 0, U3 custom1, U30 -, U31 =, U32 BackSp, U33 Ins, U34 Home, U35 PaUp, U36 Tab, U37 Q, U38 W, U39 E, U4 F1, U40 R, U41 T, U42 Y, U43 U, U44 I, U45 O, U46 P, U47 [, U48 ], U49 \, U5 F2, U50 Del, U51 End, U52 PaDo, U53 Caps, U54 A, U55 S, U56 D, U57 F, U58 G, U59 H, U6 F3, U60 J, U61 K, U62 L, U63 ;, U64 ", U65 Ent, U66 LShif, U67 Z, U68 X, U69 C, U7 F4, U70 V, U71 B, U72 N, U73 M, U74 <, U75 >, U76 ?, U77 Custom, U78 RShif, U79 ArUp, U8 F5, U80 LCrtl, U81 LSuper, U82 LAlt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

Commit message: cc
Signed-off-by: bornav <borna.vincek1@gmail.com>
Parts:
- U99: footprint waveshare:waveshare-rp2040-zero -> waveshare:waveshare-rp2040-zero_no_inner
Connections:
- net GND: now reaches U99.57 (GND)
Changed lines of the file:
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@@
+    )
+  )
+  (symbol (lib_id "power:GND") (at -144.78 246.38 0) (unit 1)
+    (in_bom yes) (on_board yes) (dnp no) (fields_autoplaced)
+    (property "Reference" "#PWR01" (at -144.78 252.73 0)
+      (effects (font (size 1.27 1.27)) hide)
+    )
+    (property "Value" "GND" (at -144.78 251.46 0)
+      (effects (font (size 1.27 1.27)))
+    )
+    (property "Footprint" "" (at -144.78 246.38 0)
+      (effects (font (size 1.27 1.27)) hide)
+    )
+    (property "Datasheet" "" (at -144.78 246.38 0)
+      (effects (font (size 1.27 1.27)) hide)
+    )
+    (pin "1")
+    (instances
+      (project "verasity_PCB"
+        (path "/eb9e929c-804a-48fb-9333-213839b64271"
+          (reference "#PWR01") (unit 1)
+        )
+      )
     )
   )
@@
       (effects (font (size 1.27 1.27)) (justify left))
     )
-    (property "Footprint" "waveshare:waveshare-rp2040-zero" (at -144.78 200.66 0)
-      (effects (font (size 1.27 1.27)) hide)
-    )
+    (property "Footprint" "waveshare:waveshare-rp2040-zero_no_inner" (at -144.78 200.66 0)
+      (effects (font (size 1.27 1.27)) hide)
+    )

Commit message: prerelease
Signed-off-by: bornav <borna.vincek1@gmail.com>
Parts:
- U99: footprint waveshare:waveshare-rp2040-zero_no_inner -> waveshare:waveshare-rp2040-pad_solder_with_cutout
Connections:
- net COL7: now also U99.2 (GPIO0); no longer U99.8 (GPIO6)
Changed lines of the file:
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@@
     (stroke (width 0) (type default))
   )
-  (wire (pts (xy -119.38 177.8) (xy -111.76 177.8))
-    (stroke (width 0) (type default))
-  )
   (wire (pts (xy -111.76 187.96) (xy -119.38 187.96))
     (stroke (width 0) (type default))
@@
     (stroke (width 0) (type default))
   )
+  (wire (pts (xy -119.38 162.56) (xy -111.76 162.56))
+    (stroke (width 0) (type default))
+  )
   (wire (pts (xy 135.89 254) (xy 135.89 262.89))
     (stroke (width 0) (type default))
@@
     )
   )
-  (global_label "COL7" (shape bidirectional) (at -111.76 177.8 0)
+  (global_label "COL7" (shape bidirectional) (at -111.76 162.56 0)
     (effects (font (size 1.27 1.27)) (justify left))
-    (property "Intersheetrefs" "${INTERSHEET_REFS}" (at -111.76 177.8 0)
+    (property "Intersheetrefs" "${INTERSHEET_REFS}" (at -111.76 162.56 0)
       (effects (font (size 1.27 1.27)) hide)
     )
@@
       (effects (font (size 1.27 1.27)) (justify left))
     )
-    (property "Footprint" "waveshare:waveshare-rp2040-zero_no_inner" (at -144.78 200.66 0)
+    (property "Footprint" "waveshare:waveshare-rp2040-pad_solder_with_cutout" (at -144.78 200.66 0)
       (effects (font (size 1.27 1.27)) hide)
     )

Commit message: new 2.1 prod
Parts:
- added H1, H2, H3, H4, H5, H6, H7, H8, H9: MountingHole_Pad, MountingHole:MountingHole_2.1mm, symbol Mechanical:MountingHole_Pad
- U32, U65, U66: footprint socket_multi_mechanical_keyboard:inverse_socket_MX_hotswap -> socket_multi_mechanical_keyboard:inverse_socket_MX_hotswap_2.5U_stabilizers
- U99: comment (none) -> RP2040-Zero
Connections:
- net COL1: now also U99.37 (GPIO25); no longer U20.1 (COL), U37.1 (COL), U54.1 (COL), U67.1 (COL), U81.1 (COL), U99.16 (GPIO13)
- net COL2: now also U20.1 (COL), U37.1 (COL), U54.1 (COL), U67.1 (COL), U81.1 (COL), U99.18 (GPIO15); no longer U21.1 (COL), U22.1 (COL), U38.1 (COL), U39.1 (COL), U4.1 (COL), U5.1 (COL), U55.1 (COL), U56.1 (COL), U68.1 (COL), U69.1 (COL), U82.1 (COL), U83.1 (COL), U99.11 (GPIO8)
- net COL3: now also U21.1 (COL), U38.1 (COL), U4.1 (COL), U55.1 (COL), U68.1 (COL), U82.1 (COL), U99.17 (GPIO14); no longer U23.1 (COL), U24.1 (COL), U40.1 (COL), U41.1 (COL), U57.1 (COL), U58.1 (COL), U6.1 (COL), U7.1 (COL), U70.1 (COL), U71.1 (COL), U84.1 (COL), U85.1 (COL), U99.38 (GPIO26_ADC0)
- net COL4: now also U22.1 (COL), U39.1 (COL), U5.1 (COL), U56.1 (COL), U69.1 (COL), U83.1 (COL), U99.16 (GPIO13); no longer U25.1 (COL), U26.1 (COL), U42.1 (COL), U43.1 (COL), U59.1 (COL), U60.1 (COL), U72.1 (COL), U73.1 (COL), U8.1 (COL), U86.1 (COL), U87.1 (COL), U9.1 (COL), U99.5 (GPIO3)
- net COL5: now also U23.1 (COL), U40.1 (COL), U57.1 (COL), U6.1 (COL), U70.1 (COL), U84.1 (COL), U99.15 (GPIO12); no longer U10.1 (COL), U11.1 (COL), U27.1 (COL), U28.1 (COL), U44.1 (COL), U45.1 (COL), U61.1 (COL), U62.1 (COL), U74.1 (COL), U75.1 (COL), U89.1 (COL), U90.1 (COL), U99.4 (GPIO2)
- net COL6: now also U24.1 (COL), U41.1 (COL), U58.1 (COL), U7.1 (COL), U71.1 (COL), U85.1 (COL), U99.14 (GPIO11); no longer U12.1 (COL), U13.1 (COL), U29.1 (COL), U30.1 (COL), U46.1 (COL), U47.1 (COL), U63.1 (COL), U64.1 (COL), U76.1 (COL), U77.1 (COL), U91.1 (COL), U92.1 (COL), U99.3 (GPIO1)
- net COL7: now also U25.1 (COL), U42.1 (COL), U59.1 (COL), U72.1 (COL), U8.1 (COL), U86.1 (COL), U99.13 (GPIO10); no longer U14.1 (COL), U15.1 (COL), U16.1 (COL), U3.1 (COL), U31.1 (COL), U32.1 (COL), U33.1 (COL), U48.1 (COL), U49.1 (COL), U50.1 (COL), U65.1 (COL), U78.1 (COL), U93.1 (COL), U97.1 (COL), U99.2 (GPIO0)
- net COL8: now also U26.1 (COL), U43.1 (COL), U60.1 (COL), U73.1 (COL), U87.1 (COL), U9.1 (COL), U99.12 (GPIO9); no longer U17.1 (COL), U18.1 (COL), U34.1 (COL), U35.1 (COL), U51.1 (COL), U52.1 (COL), U79.1 (COL), U88.1 (COL), U94.1 (COL), U95.1 (COL), U96.1 (COL), U98.1 (COL), U99.9 (GPIO7)
- net ROW1: now also U99.36 (GPIO24); no longer U99.6 (GPIO4)
- net ROW2: now also U99.38 (GPIO26_ADC0); no longer U99.13 (GPIO10)
- net ROW3: now also U99.39 (GPIO27_ADC1); no longer U99.12 (GPIO9)
- net ROW4: now also U99.40 (GPIO28_ADC2); no longer U99.7 (GPIO5)
- net ROW5: now also U99.35 (GPIO23); no longer U99.17 (GPIO14)
- net ROW6: now also U99.41 (GPIO29_ADC3); no longer U99.39 (GPIO27_ADC1)
- net COL11: now reaches U99.8 (GPIO6)
- net COL11: now also U12.1 (COL), U29.1 (COL), U46.1 (COL), U63.1 (COL), U76.1 (COL), U91.1 (COL)
- new net COL10: U11.1 (COL), U28.1 (COL), U45.1 (COL), U62.1 (COL), U75.1 (COL), U90.1 (COL), U99.9 (GPIO7)
- new net COL12: U13.1 (COL), U30.1 (COL), U47.1 (COL), U64.1 (COL), U77.1 (COL), U92.1 (COL), U99.7 (GPIO5)
- new net COL13: U14.1 (COL), U31.1 (COL), U48.1 (COL), U65.1 (COL), U78.1 (COL), U99.6 (GPIO4)
- new net COL14: U15.1 (COL), U32.1 (COL), U49.1 (COL), U99.5 (GPIO3)
- new net COL15: U16.1 (COL), U3.1 (COL), U33.1 (COL), U50.1 (COL), U93.1 (COL), U97.1 (COL), U99.4 (GPIO2)
- new net COL16: U17.1 (COL), U34.1 (COL), U51.1 (COL), U79.1 (COL), U88.1 (COL), U94.1 (COL), U99.3 (GPIO1)
- new net COL17: U18.1 (COL), U35.1 (COL), U52.1 (COL), U95.1 (COL), U96.1 (COL), U98.1 (COL), U99.2 (GPIO0)
- new net COL9: U10.1 (COL), U27.1 (COL), U44.1 (COL), U61.1 (COL), U74.1 (COL), U89.1 (COL), U99.11 (GPIO8)
Other:
- moved on the sheet: U99
